File: Kicad_schematics/testbench_io/testbench_io.sch (KiCad schematic (older format))
At the start: 47 parts

Commit message: added hierarchical sheets
Signed-off-by: Mojitas <47667093+Mojitas@users.noreply.github.com>
Parts:
- removed Q? (x4): BUK9M42-60EX, Package_TO_SOT_SMD:LFPAK33, symbol Transistor_FET:BUK9M42-60EX
- removed R? (x4): R_Small, symbol Device:R_Small
- gave numbers to parts that had none: 39
Connections:
- net labels removed: Brake_acti, Brake_lights, Front_acti, Front_lights, Left_acti, Left_indicator, Right_acti, Right_indicator
- wire segments 186 -> 162
Other:
- moved on the sheet: D1, D2, D3, D4, D5, J1, R1, R2, R3, R4, R5, R8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
