File: Kicad_schematics/testbench_io/testbench_io.kicad_pcb (KiCad board)
At the start: 2 copper layers, 183 x 130 mm, 75 parts, among them J101 Conn_01x02, J102 Conn_01x02, J103 Conn_01x02, J104 DB37_Female_MountingHoles, J301 Conn_01x04, J302 Conn_01x04, J303 Conn_01x04, Q201 2N3904, Q301 IPD50R380CE, Q302 IPD50R380CE, Q303 IPD50R380CE, Q304 IPD50R380CE, Q305 IPD50R380CE, Q306 IPD50R380CE, SW101 SW_SPST, SW102 SW_Push, SW103 SW_Push, SW104 SW_Push, SW105 SW_Push, SW106 SW_SPST, SW107 SW_SPST, SW108 SW_DIP_x08, SW109 SW_SPST, SW110 SW_Push, SW111 SW_SPST, SW112 SW_SPST, SW113 SW_SPST, SW114 SW_DPDT_x2, SW201 SW_DIP_x01, U101 NUCLEO64-F476RG, U102 CJMCU_MCP2551, U201 PCF8574AN

Commit message: PCB sent to board house
Parts:
- J104: footprint Connector_Dsub:DSUB-37_Female_Horizontal_P2.77x2.84mm_EdgePinOffset7.70mm_Housed_MountingHolesOffset9.12mm -> Solar_team:Wuerth__angeled_dsub_37_618037231321
- moved J104 28.2 mm to (159.0, 145.9)
Routing:
- net GND: track 792.2 -> 808.4 mm
- net /TRM_14: track 27.8 -> 38.2 mm
- net /TRM_15: track 52.9 -> 59.4 mm
- net Net-(J102-Pad2): track 79.6 -> 84.4 mm
- net /TRM_7: track 50.1 -> 54.9 mm
- net /TRM_01: track 74.6 -> 79.3 mm
- net TRM_GND: track 68.3 -> 72.9 mm
- net /TRM_25: track 46.7 -> 51.2 mm
- net /TRM_20: track 73.8 -> 78.4 mm
- net /TRM_05: track 36.9 -> 41.5 mm
- net /TRM_06: track 38.3 -> 42.8 mm
- net /TRM_22: track 42.3 -> 46.8 mm
- net /TRM_02: track 57.0 -> 61.5 mm
- net TRM_VDD: track 66.3 -> 70.2 mm
- net Net-(J102-Pad1): track 83.7 -> 85.8 mm
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Other:
- rule trace_min: 0.2 -> 0.127
- rule via_min_size: 0.4 -> 0.6
