File: Kicad_schematics/testbench_io/CAN.sch (KiCad schematic (older format))
At the start: 4 parts, among them J601 Conn_01x02, U601 CJMCU_MCP2551

Commit message: fixes
Parts:
- removed JP601: SolderJumper_2_Open, Jumper:SolderJumper-2_P1.3mm_Open_Pad1.0x1.5mm, symbol Jumper:SolderJumper_2_Open
Connections:
- net CAN_N: now reaches J601.1 (Pin_1), R601.1, U601.6 (CAN_L-)
- net CAN_N: no longer J601.2 (Pin_2), U601.5 (CAN_H+)
- net CAN_P: now reaches R601.2
- net CAN_P: now also J601.2 (Pin_2), U601.5 (CAN_H+)
Other:
- moved on the sheet: J601, R601
Changed lines of the file:
@@
 $Descr A4 11693 8268
 encoding utf-8
-Sheet 7 7
+Sheet 6 7
 Title ""
 Date ""
@@
 L Connector_Generic:Conn_01x02 J?
 U 1 1 605E666D
-P 6600 3550
+P 6850 3650
 AR Path="/605E666D" Ref="J?"  Part="1"
 AR Path="/605E5633/605E666D" Ref="J601"  Part="1"
-F 0 "J601" H 6680 3542 50  0000 L CNN
-F 1 "Conn_01x02" H 6680 3451 50  0000 L CNN
-F 2 "Connector_JST:JST_XH_S2B-XH-A_1x02_P2.50mm_Horizontal" H 6600 3550 50  0001 C CNN
-F 3 "~" H 6600 3550 50  0001 C CNN
-	1    6600 3550
-	1    0    0    -1
+F 0 "J601" H 6930 3642 50  0000 L CNN
+F 1 "Conn_01x02" H 6930 3551 50  0000 L CNN
+F 2 "Connector_JST:JST_XH_S2B-XH-A_1x02_P2.50mm_Horizontal" H 6850 3650 50  0001 C CNN
+F 3 "~" H 6850 3650 50  0001 C CNN
+	1    6850 3650
+	1    0    0    1
 $EndComp
 Wire Wire Line
-	6350 3550 6400 3550
-Wire Wire Line
-	6150 4000 6150 3950
-Wire Wire Line
-	6350 4000 6350 3950
-Connection ~ 6350 3550
-Wire Wire Line
-	6350 3650 6350 3550
+	6150 4200 6150 4150
 Connection ~ 6150 3650
 Wire Wire Line
-	6150 3750 6150 3650
-Wire Wire Line
-	6100 3550 6350 3550
-$Comp
-L Jumper:SolderJumper_2_Open JP?
-U 1 1 605E667B
-P 6350 3800
-AR Path="/605E667B" Ref="JP?"  Part="1"
-AR Path="/605E5633/605E667B" Ref="JP601"  Part="1"
-F 0 "JP601" V 6304 3868 50  0000 L CNN
-F 1 "SolderJumper_2_Open" V 6395 3868 50  0000 L CNN
-F 2 "Jumper:SolderJumper-2_P1.3mm_Open_Pad1.0x1.5mm" H 6350 3800 50  0001 C CNN
-F 3 "~" H 6350 3800 50  0001 C CNN
-	1    6350 3800
-	0    1    1    0
-$EndComp
+	6150 3950 6150 3650
 Wire Wire Line
 	6100 3650 6150 3650
@@
 GND_MCU
 Wire Wire Line
-	6150 4000 6350 4000
+	6150 4200 6350 4200
 $Comp
 L Device:R_Small R?
 U 1 1 605E6686
-P 6150 3850
+P 6150 4050
 AR Path="/605E6686" Ref="R?"  Part="1"
 AR Path="/605E5633/605E6686" Ref="R601"  Part="1"
-F 0 "R601" V 6250 3850 50  0000 C CNN
-F 1 "120" V 6050 3850 50  0000 C CNN
-F 2 "Resistor_SMD:R_0603_1608Metric" H 6150 3850 50  0001 C CNN
-F 3 "~" H 6150 3850 50  0001 C CNN
-	1    6150 3850
+F 0 "R601" V 6250 4050 50  0000 C CNN
+F 1 "120" V 6050 4050 50  0000 C CNN
+F 2 "Resistor_SMD:R_0603_1608Metric" H 6150 4050 50  0001 C CNN
+F 3 "~" H 6150 4050 50  0001 C CNN
+	1    6150 4050
 	1    0    0    -1
 $EndComp
 Wire Wire Line
 	5350 3850 5400 3850
-$Comp
-L Solarteam:CJMCU_MCP2551 U?
-U 1 1 605E668D
-P 5750 3600
-AR Path="/605E668D" Ref="U?"  Part="1"
-AR Path="/605E5633/605E668D" Ref="U601"  Part="1"
-F 0 "U601" H 5600 3600 50  0000 C CNN
-F 1 "CJMCU_MCP2551" H 5750 3950 50  0000 C CNN
-F 2 "Solar_team:CJMCU_2551" H 5750 3600 50  0001 C CNN
-F 3 "" H 5750 3600 50  0001 C CNN
-	1    5750 3600
-	1    0    0    -1
-$EndComp
-Wire Wire Line
-	6150 3650 6350 3650
-Connection ~ 6350 3650
-Wire Wire Line
-	6350 3650 6400 3650
 Wire Notes Line
 	7300 3200 7300 4250
@@
 Text HLabel 5300 3450 0    50   Input ~ 0
 CTX
+Text Label 6600 3550 1    50   ~ 0
+CAN_P
+Text Label 6600 3650 3    50   ~ 0
+CAN_N
+Wire Wire Line
+	6150 3650 6650 3650
+Wire Wire Line
+	6100 3550 6350 3550
+Connection ~ 6350 3550
+Wire Wire Line
+	6350 3550 6650 3550
+$Comp
+L Solarteam:CJMCU_MCP2551 U601
+U 1 1 60350ACB
+P 5750 3600
+F 0 "U601" H 5750 4075 50  0000 C CNN
+F 1 "CJMCU_MCP2551" H 5750 3984 50  0000 C CNN
+F 2 "Solar_team:CJMCU_2551" H 5750 3600 50  0001 C CNN
+F 3 "" H 5750 3600 50  0001 C CNN
+	1    5750 3600
+	1    0    0    -1
+$EndComp
+Wire Wire Line
+	6350 3550 6350 4200
 $EndSCHEMATC
