File: Kicad_schematics/testbench_io/MCU_IO.sch (KiCad schematic (older format))
At the start: 20 parts, among them SW401 SW_Push, SW402 SW_Push, SW403 SW_Push, SW404 SW_Push, SW405 SW_SPST, SW406 SW_SPST, SW407 SW_Push, SW408 SW_DPDT_x2

Commit message: fixes
Parts:
- SW405, SW406: footprint Solar_team:RND-Slide-Switch -> Solar_team:MFP120
- SW408: footprint Solar_team:RND-Slide-Switch -> Solar_team:MFP130
Changed lines of the file:
@@
 F 0 "SW408" H 7400 3385 50  0000 C CNN
 F 1 "SW_DPDT_x2" H 7400 3294 50  0000 C CNN
-F 2 "Solar_team:RND-Slide-Switch" H 7400 3100 50  0001 C CNN
+F 2 "Solar_team:MFP130" H 7400 3100 50  0001 C CNN
 F 3 "~" H 7400 3100 50  0001 C CNN
 	1    7400 3100
@@
 F 0 "SW406" H 6800 3935 50  0000 C CNN
 F 1 "SW_SPST" H 6800 3844 50  0000 C CNN
-F 2 "Solar_team:RND-Slide-Switch" H 6800 3700 50  0001 C CNN
+F 2 "Solar_team:MFP120" H 6800 3700 50  0001 C CNN
 F 3 "~" H 6800 3700 50  0001 C CNN
 	1    6800 3700
@@
 F 0 "SW405" H 6800 3585 50  0000 C CNN
 F 1 "SW_SPST" H 6800 3494 50  0000 C CNN
-F 2 "Solar_team:RND-Slide-Switch" H 6800 3350 50  0001 C CNN
+F 2 "Solar_team:MFP120" H 6800 3350 50  0001 C CNN
 F 3 "~" H 6800 3350 50  0001 C CNN
 	1    6800 3350
